File: firstpcb.kicad_pcb (KiCad board)
At the start: 2 copper layers, 6.3 x 6.3 mm, 24 parts, among them SW1 SW_Push, U1 ATmega32U4-AU, Y1 16MHz

Commit message: 0
Parts:
- F1, R2, R3, R4, SW1, USB1: moved to B.Cu
- moved SW1 64.7 mm to (108.7, 131.8), turned to 180 degrees
- moved R4 63.8 mm to (137.3, 123.0), turned to 90 degrees
- moved R1 49.1 mm to (118.3, 108.0)
- moved R2 48.7 mm to (111.9, 109.5), turned to 90 degrees
- moved C6 46.0 mm to (132.6, 127.8)
- moved C7 46.0 mm to (123.0, 127.8)
- moved U1 46.0 mm to (127.8, 118.3)
- moved C5 45.5 mm to (137.3, 112.7)
- moved C1 44.9 mm to (131.8, 104.0)
- moved C2 44.9 mm to (123.8, 104.0)
- moved Y1 44.9 mm to (127.8, 104.0)
- moved C3 44.4 mm to (116.7, 119.1)
- moved USB1 41.9 mm to (110.3, 99.2), turned to 270 degrees
- moved C4 39.8 mm to (121.4, 108.0), turned to 90 degrees
- moved R3 38.5 mm to (108.7, 109.5), turned to 90 degrees
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Connections:
- U1 pad 27: Net-(U1-Pad27) -> ROW0
- U1 pad 28: Net-(U1-Pad28) -> COL0
- U1 pad 29: Net-(U1-Pad29) -> COL1
- U1 pad 30: Net-(U1-Pad30) -> ROW1
- USB1 pad 3: Net-(USB1-Pad3) -> D+
- USB1 pad 5: D+ -> VCC
- USB1 pad 6: VCC -> Net-(USB1-Pad6)
Other:
- board size 6.3 x 6.3 mm -> 75.4 x 38.1 mm
